Commit message: Bugfix: Vehicle visualization missing

File: AD-EYE/Data/URDF_Actor_Models/BMW_X5/default.urdf (robot description, URDF)
Before this commit: robot car, 1 links, 0 joints
Links:
- link base_link: geometry visual mesh filename=file:///home/naveenm/AD-EYE-WASP/AD-EYE/Data/URDF_Actor_Mod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 scale=0.03 0.03 0.03

Commit message: Fixed hardcoded paths in actor model, localization launch and unittest files

File: AD-EYE/Data/URDF_Actor_Models/BMW_X5/default.urdf (robot description, URDF)
Before this commit: robot car, 1 links, 0 joints
Links:
- link base_link: geometry visual mesh filename=file://$(find adeye)/../../../../AD-EYE/Data/URDF_Actor_Mod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 scale=0.03 0.03 0.03

Commit message: Changed model to package rather than file relative path

File: AD-EYE/Data/URDF_Actor_Models/BMW_X5/default.urdf (robot description, URDF)
Before this commit: robot car, 1 links, 0 joints
Links:
- link base_link: geometry visual mesh filename=package://adeye/../../../../AD-EYE/Data/URDF_Actor_Models/B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 scale=0.03 0.03 0.03

Commit message: Changed gps coordinates for initial pose

File: AD-EYE/Data/URDF_Actor_Models/BMW_X5/default.urdf (robot description, URDF)
Before this commit: robot car, 1 links, 0 joints
Links:
- added link os_sensor
Joints:
- added joint base_link_to_sensor_joint: type fixed, parent base_link, child os_sensor, origin xyz=0.0 0.0 0.0 rpy=0 0 0
